Commit message: changes names

File: src/qube_description/urdf/qube.macro.xacro (robot description, xacro)
@@ -1,4 +1,4 @@
 <?xml version="1.0"?>
-<robot xmlns:xacro="http://www.ros.org/wiki/xacro">
+<robot xmlns:xacro="http://www.ros.org/wiki/xacro" >
   <material name="blue">
       <color rgba="0 0 0.8 1"/>
@@ -10,5 +10,5 @@
       <color rgba="1 1 1 1"/>
   </material>
-  <xacro:macro name="simple_motor" params="parent prefix">
+  <xacro:macro name="qube" params="parent prefix">
     <xacro:property name="box_width" value="0.102"/>
     <xacro:property name="rotor_radius" value="0.025"/>

File: src/qube_description/urdf/qube.urdf.xacro (robot description, xacro)
@@ -1,5 +1,5 @@
 <?xml version="1.0"?>
 <robot xmlns:xacro="http://www.ros.org/wiki/xacro" name="myfirst">
-  <xacro:include filename="$(find joint_description)/urdf/joint_model.macro.urdf"/>
+  <xacro:include filename="$(find qube_description)/urdf/qube.macro.xacro"/>
   <link name="world"/>
   <link name="base_link"/>
@@ -14,5 +14,5 @@
     <origin xyz="2 0 0" />
   </joint>
-  <xacro:simple_motor parent="base_link" prefix="motor1_"/>
-  <xacro:simple_motor parent="base_link2" prefix="motor2_"/>
+  <xacro:qube parent="base_link" prefix="motor1_"/>
+  <xacro:qube parent="base_link2" prefix="motor2_"/>
 </robot>

Commit message: Fixed macro

File: src/qube_description/urdf/qube.macro.xacro (robot description, xacro)
@@ -43,5 +43,5 @@
       <origin xyz="0 0 ${box_width/2}"/>
     </joint>
-    <joint name="${prefix}angle_joint" type="revolute">
+    <joint name="${prefix}motor_joint" type="revolute">
       <parent link="${prefix}stator_link"/>
       <child link="${prefix}rotor_link"/>

Commit message: Small changes

File: src/qube_description/urdf/qube.macro.xacro (robot description, xacro)
@@ -1,7 +1,4 @@
 <?xml version="1.0"?>
 <robot xmlns:xacro="http://www.ros.org/wiki/xacro" >
-  <material name="blue">
-      <color rgba="0 0 0.8 1"/>
-    </material>
     <material name="black">
       <color rgba="0 0 0 1"/>
@@ -11,4 +8,5 @@
   </material>
   <xacro:macro name="qube" params="parent prefix">
+    <!--Dimensions of Qube-->
     <xacro:property name="box_width" value="0.102"/>
     <xacro:property name="rotor_radius" value="0.025"/>
